Commit message: Real robot simulation

File: description/robot.urdf.xacro (robot description, xacro)
@@ -2,4 +2,7 @@
 <robot xmlns:xacro="http://www.ros.org/wiki/xacro"  name="robot">
     <xacro:include filename="robot_core.xacro"/>
-    <xacro:include filename="gazebo_control.xacro"/>
+    <!-- <xacro:include filename="gazebo_control.xacro"/>-->
+    <xacro:include filename="lidar.xacro"/>
+    <xacro:include filename="camera.xacro"/>
+    <xacro:include filename="ros2_control.xacro"/>
 </robot>

File: description/robot_core.xacro (robot description, xacro)
@@ -2,4 +2,18 @@
 <robot xmlns:xacro="http://www.ros.org/wiki/xacro">
     <xacro:include filename="inertial_macros.xacro"/>
+    <xacro:property name="chassis_length" value="0.20" />
+    <xacro:property name="chassis_width" value="0.20" />
+    <xacro:property name="chassis_height" value="0.13" />
+    <xacro:property name="chassis_mass" value="1.0" />
+    <xacro:property name="wheel_radius" value="0.032" />
+    <xacro:property name="wheel_thickness" value="0.026" />
+    <xacro:property name="wheel_mass" value="0.5" />
+    <xacro:property name="wheel_offset_x" value="0.226" />
+    <xacro:property name="wheel_offset_y" value="0.113" />
+    <xacro:property name="wheel_offset_z" value="${wheel_radius}" />
+    <xacro:property name="caster_wheel_radius" value="0.03" />
+    <xacro:property name="caster_wheel_mass" value="0.01" />
+    <xacro:property name="caster_wheel_offset_x" value="0.06" />
+    <xacro:property name="caster_wheel_offset_z" value="-${chassis_height/2}" />
     <!-- MATERIALS -->
     <material name="white">
@@ -13,8 +27,11 @@
     </material>
     <material name="black">
-        <color rgba="0 0 0 1 " />
+        <color rgba="0 0 0 1 " />-
+    </material>
+    <material name="red">
+        <color rgba="1 0 0 1 " />
     </material>
     <!-- BASE LINK-->
-    <link name="base_link">
+    <link name="base_link">0
     </link>
     <!-- CHASSIS-->
@@ -22,18 +39,18 @@
         <parent link="base_link"/>
         <child link="chassis"/>
-        <origin xyz="-0.1 0 0" />
+        <origin xyz="0.04 0 ${chassis_height/2 + wheel_radius}" />
     </joint>
+z
     <link name="chassis">
         <visual>
-            <origin xyz="0.15 0 0.075" />
             <geometry>
-                <box size="0.3 0.3 0.15"/>
+                <box size="0.20 0.20 0.13"/>
             </geometry>
-            <material name="white"/>
+            <material name="black"/>
         </visual>
         <collision>
-            <origin xyz="0.15 0 0.075" />
+            <origin xyz="0 0 0" />
             <geometry>
-                <box size="0.3 0.3 0.15"/>
+                <box size="0.20 0.20 0.13"/>
             </geometry>
         </collision>
@@ -43,9 +60,9 @@
     </link>
     <gazebo reference="chassis">
-        <material>Gazebo/White</material>
+        <material>Gazebo/Black</material>
     </gazebo>
     <!-- LEFT WHEEL LINK-->
     <joint name="left_wheel_joint" type="continuous">
-        <origin xyz="0 0.175 0.0" rpy="-${pi/2} 0 0"/>
+        <origin xyz="0 ${wheel_offset_y} ${wheel_offset_z}" rpy="-${pi/2} 0 0"/>
         <parent link="base_link"/>
         <child link="left_wheel"/>
@@ -55,5 +72,5 @@
         <visual>
             <geometry>
-                <cylinder radius="0.05" length="0.04"/>
+                <cylinder radius="${wheel_radius}" length="${wheel_thickness}"/>
             </geometry>
             <material name="blue"/>
@@ -61,8 +78,8 @@
         <collision>
             <geometry>
-                <cylinder radius="0.05" length="0.04"/>
+                <cylinder radius="${wheel_radius}" length="${wheel_thickness}"/>
             </geometry>
         </collision>
-        <xacro:inertial_cylinder mass="0.1" length="0.04" radius="0.05">
+        <xacro:inertial_cylinder mass="${wheel_mass}" length="${wheel_thickness}" radius="${wheel_radius}">
             <origin xyz="0 0 0" rpy="0 0 0"/>
         </xacro:inertial_cylinder>
@@ -73,5 +90,5 @@
     <!-- RIGHT WHEEL LINK-->
     <joint name="right_wheel_joint" type="continuous">
-        <origin xyz="0 -0.175 0.0" rpy="${pi/2} 0 0"/>
+        <origin xyz="0 -${wheel_offset_y} ${wheel_offset_z}" rpy="${pi/2} 0 0"/>
         <parent link="base_link"/>
         <child link="right_wheel"/>
@@ -81,5 +98,5 @@
         <visual>
             <geometry>
-                <cylinder radius="0.05" length="0.04"/>
+                <cylinder radius="${wheel_radius}" length="${wheel_thickness}"/>
             </geometry>
             <material name="blue"/>
@@ -87,8 +104,8 @@
         <collision>
             <geometry>
-                <cylinder radius="0.05" length="0.04"/>
+                <cylinder radius="${wheel_radius}" length="${wheel_thickness}"/>
             </geometry>
         </collision>
-        <xacro:inertial_cylinder mass="0.1" length="0.04" radius="0.05">
+        <xacro:inertial_cylinder mass="${wheel_mass}" length="${wheel_thickness}" radius="${wheel_radius}">
             <origin xyz="0 0 0" rpy="0 0 0"/>
         </xacro:inertial_cylinder>
@@ -101,24 +118,24 @@
         <parent link="chassis"/>
         <child link="caster_wheel"/>
-        <origin xyz="0.24 0 0"/>
+        <origin xyz="${caster_wheel_offset_x} 0 ${caster_wheel_offset_z}"/>
     </joint>
     <link name="caster_wheel">
         <visual>
             <geometry>
-                <sphere radius="0.05"/>
+                <sphere radius="${caster_wheel_radius}"/>
             </geometry>
-            <material name="black"/>
+            <material name="blue"/>
         </visual>
         <collision>
             <geometry>
-                <sphere radius="0.05"/>
+                <sphere radius="${caster_wheel_radius}"/>
             </geometry>
         </collision>
-        <xacro:inertial_sphere mass="0.1" radius="0.05">
+        <xacro:inertial_sphere mass="${caster_wheel_mass}" radius="${caster_wheel_radius}">
             <origin xyz="0 0 0" rpy="0 0 0"/>
         </xacro:inertial_sphere>
     </link>
     <gazebo reference="caster_wheel">
-        <material>Gazebo/Black</material>
+        <material>Gazebo/Blue</material>
         <mu1 value="0.0001"/>
         <mu2 value="0.0001"/>
