Commit message: preparing for ros remote

File: description/camera.xacro (robot description, xacro)
@@ -4,5 +4,5 @@
         <parent link="chassis"/>
         <child link="camera_link"/>
-        <origin xyz="${chassis_length/2} 0 0" rpy="0 0 0"/>
+        <origin xyz="${chassis_length/2-0.005} 0 0.045" rpy="0 0 0"/>
     </joint>
     <link name="camera_link">

File: description/lidar.xacro (robot description, xacro)
@@ -4,5 +4,5 @@
         <parent link="chassis"/>
         <child link="laser_frame"/>
-        <origin xyz="0 0 0.065" rpy="0 0 0"/>
+        <origin xyz="0.08 0 0.065" rpy="0 0 0"/>
     </joint>
     <link name="laser_frame">

File: description/robot.urdf.xacro (robot description, xacro)
@@ -3,6 +3,6 @@
     <xacro:include filename="robot_core.xacro"/>
     <!-- <xacro:include filename="gazebo_control.xacro"/>-->
-    <xacro:include filename="lidar.xacro"/>
-    <xacro:include filename="camera.xacro"/>
+    <!--<xacro:include filename="lidar.xacro"/>-->
+    <!--<xacro:include filename="camera.xacro"/>-->
     <xacro:include filename="ros2_control.xacro"/>
 </robot>

File: description/robot_core.xacro (robot description, xacro)
@@ -1,20 +1,177 @@
 <?xml version="1.0"?>
 <robot xmlns:xacro="http://www.ros.org/wiki/xacro">
+    <link name="base_link">
+    </link>
+    <link name="base_footprint">
+    </link>
+    <link name="camera_link">
+      <inertial>
+        <origin xyz="0 0 0" rpy="0 0 0"/>
+        <mass value="2.0"/>
+        <inertia ixx="1.25714" ixy="0" ixz="0" iyy="0.71958" iyz="0" izz="0.71958"/>
+      </inertial>
+      <visual name="camera">
+        <origin xyz="0 0 0" rpy="0 0 0"/>
+        <geometry>
+          <mesh filename="file:///home/dev/dev_ws/install/rover/share/rover/meshes/stl/Cube.006.stl" scale="1.0 1.0 1.0"/>
+        </geometry>
+      </visual>
+      <collision name="camera">
+        <origin xyz="0 0 0" rpy="0 0 -3.14159"/>
+        <geometry>
+          <mesh filename="file:///home/dev/dev_ws/install/rover/share/rover/meshes/stl/Cube.028.stl" scale="1.0 1.0 1.0"/>
+        </geometry>
+      </collision>
+    </link>
+    <link name="caster_link">
+      <inertial>
+        <origin xyz="0 0 0" rpy="0 0 0"/>
+        <mass value="1.0"/>
+        <inertia ixx="2e-05" ixy="0" ixz="0" iyy="2e-05" iyz="0" izz="2e-05"/>
+      </inertial>
+      <visual name="caster">
+        <origin xyz="0 0 0" rpy="0 0 0"/>
+        <geometry>
+          <mesh filename="file:///home/dev/dev_ws/install/rover/share/rover/meshes/stl/CasterBallWheel001.stl" scale="1.0 1.0 1.0"/>
+        </geometry>
+      </visual>
+      <collision name="caster">
+        <origin xyz="0 0 -0.00023" rpy="0 0 -3.14159"/>
+        <geometry>
+          <mesh filename="file:///home/dev/dev_ws/install/rover/share/rover/meshes/stl/CasterBallWheel001.002.stl" scale="1.0 1.0 1.0"/>
+        </geometry>
+      </collision>
+    </link>
+    <link name="chassis_link">
+      <inertial>
+        <origin xyz="-0.00047 0 -0.00023" rpy="0 0 0"/>
+        <mass value="2.0"/>
+        <inertia ixx="83.98086" ixy="0" ixz="0" iyy="93.54912" iyz="0" izz="149.48003"/>
+      </inertial>
+      <visual name="chassis_link">
+        <origin xyz="0 0 0" rpy="0 0 0"/>
+        <geometry>
+          <mesh filename="file:///home/dev/dev_ws/install/rover/share/rover/meshes/stl/Cube.005.stl" scale="1.0 1.0 1.0"/>
+        </geometry>
+      </visual>
+      <collision name="chassis_link">
+        <origin xyz="-0.00047 0 -0.00023" rpy="0 0 -3.14159"/>
+        <geometry>
+          <mesh filename="file:///home/dev/dev_ws/install/rover/share/rover/meshes/stl/Cube.027.stl" scale="1.0 1.0 1.0"/>
+        </geometry>
+      </collision>
+    </link>
+    <link name="laser_frame">
+      <inertial>
+        <origin xyz="-0.00026 0 -0.00026" rpy="0 0 0"/>
+        <mass value="2.0"/>
+        <inertia ixx="18.59151" ixy="0" ixz="0" iyy="18.59446" iyz="0" izz="17.12676"/>
+      </inertial>
+      <visual name="lidar">
+        <origin xyz="0 0 0" rpy="0 0 0"/>
+        <geometry>
+          <mesh filename="file:///home/dev/dev_ws/install/rover/share/rover/meshes/stl/Cube.007.stl" scale="1.0 1.0 1.0"/>
+        </geometry>
+      </visual>
+      <collision name="lidar">
+        <origin xyz="-0.00052 0 0" rpy="0 0 -3.14159"/>
+        <geometry>
+          <mesh filename="file:///home/dev/dev_ws/install/rover/share/rover/meshes/stl/Cube.029.stl" scale="1.0 1.0 1.0"/>
+        </geometry>
+      </collision>
+    </link>
+    <link name="wheel_left_link">
+      <inertial>
+        <origin xyz="0 0 0" rpy="0 0 0"/>
+        <mass value="2.0"/>
+        <inertia ixx="12.23232" ixy="0" ixz="0" iyy="2e-05" iyz="0" izz="2e-05"/>
+      </inertial>
+      <visual name="wheel_left">
+        <origin xyz="0 0 0" rpy="0 0 0"/>
+        <geometry>
+          <mesh filename="file:///home/dev/dev_ws/install/rover/share/rover/meshes/stl/Cylinder.004.stl" scale="1.0 1.0 1.0"/>
+        </geometry>
+      </visual>
+      <collision name="wheel_left">
+        <origin xyz="0 0 0" rpy="0 0 -3.14159"/>
+        <geometry>
+          <mesh filename="file:///home/dev/dev_ws/install/rover/share/rover/meshes/stl/Cylinder.011.stl" scale="1.0 1.0 1.0"/>
+        </geometry>
+      </collision>
+    </link>
+    <link name="wheel_right_link">
+      <inertial>
+        <origin xyz="0 0 0" rpy="0 0 0"/>
+        <mass value="2.0"/>
+        <inertia ixx="12.23224" ixy="0" ixz="0" iyy="2e-05" iyz="0" izz="2e-05"/>
+      </inertial>
+      <visual name="wheel_right">
+        <origin xyz="0 0 0" rpy="0 0 0"/>
+        <geometry>
+          <mesh filename="file:///home/dev/dev_ws/install/rover/share/rover/meshes/stl/Cylinder.001.stl" scale="1.0 1.0 1.0"/>
+        </geometry>
+      </visual>
+      <collision name="wheel_right">
+        <origin xyz="0 0 0" rpy="0 0 -3.14159"/>
+        <geometry>
+          <mesh filename="file:///home/dev/dev_ws/install/rover/share/rover/meshes/stl/Cylinder.013.stl" scale="1.0 1.0 1.0"/>
+        </geometry>
+      </collision>
+    </link>
+    <joint name="base_footprint_joint" type="fixed">
+        <parent link="base_link"/>
+        <child link="base_footprint"/>
+        <origin xyz="0 0 0" rpy="0 0 0"/>
+    </joint>
+    <joint name="chassis_joint" type="fixed">
+        <parent link="base_link"/>
+        <child link="chassis_link"/>
+        <origin xyz="0 0 0" />
+    </joint>
+    <joint name="camera_joint" type="fixed">
+      <origin xyz="0.09505 0 0.06038" rpy="0 0 0"/>
+      <parent link="chassis_link"/>
+      <child link="camera_link"/>
+    </joint>
+    <joint name="caster_joint" type="fixed">
+      <origin xyz="-0.12115 0 -0.01063" rpy="0 0 0"/>
+      <parent link="chassis_link"/>
+      <child link="caster_link"/>
+    </joint>
+    <joint name="laser_joint" type="fixed">
+      <origin xyz="-0.00198 0 0.14437" rpy="0 0 0"/>
+      <parent link="chassis_link"/>
+      <child link="laser_frame"/>
+    </joint>
+    <joint name="wheel_left_joint" type="continuous">
+      <origin xyz="0.01871 0.09783 0.01952" rpy="0 0 0"/>
+      <parent link="chassis_link"/>
+      <child link="wheel_left_link"/>
+      <axis xyz="0 1.0 0"/>
+      <limit effort="0" velocity="0"/>
+    </joint>
+    <joint name="wheel_right_joint" type="continuous">
+      <origin xyz="0.01871 -0.09721 0.01952" rpy="-${pi} 0 0"/>
+      <parent link="chassis_link"/>
+      <child link="wheel_right_link"/>
+      <axis xyz="0 -1.0 0"/>
+      <limit effort="0" velocity="0"/>
+    </joint>
+<!--
     <xacro:include filename="inertial_macros.xacro"/>
-    <xacro:property name="chassis_length" value="0.20" />
-    <xacro:property name="chassis_width" value="0.20" />
-    <xacro:property name="chassis_height" value="0.13" />
+    <xacro:property name="chassis_length" value="0.304" />
+    <xacro:property name="chassis_width" value="0.304" />
+    <xacro:property name="chassis_height" value="0.065" />
     <xacro:property name="chassis_mass" value="1.0" />
-    <xacro:property name="wheel_radius" value="0.032" />
-    <xacro:property name="wheel_thickness" value="0.026" />
+    <xacro:property name="wheel_radius" value="0.045" />
+    <xacro:property name="wheel_thickness" value="0.012" />
     <xacro:property name="wheel_mass" value="0.5" />
-    <xacro:property name="wheel_offset_x" value="0.226" />
-    <xacro:property name="wheel_offset_y" value="0.113" />
+    <xacro:property name="wheel_offset_x" value="0.8" />
+    <xacro:property name="wheel_offset_y" value="${chassis_width/2+wheel_thickness*2}" />
     <xacro:property name="wheel_offset_z" value="${wheel_radius}" />
     <xacro:property name="caster_wheel_radius" value="0.03" />
-    <xacro:property name="caster_wheel_mass" value="0.01" />
-    <xacro:property name="caster_wheel_offset_x" value="0.06" />
+    <xacro:property name="caster_wheel_mass" value="1.0" />
+    <xacro:property name="caster_wheel_offset_x" value="-0.1" />
     <xacro:property name="caster_wheel_offset_z" value="-${chassis_height/2}" />
-    <!-- MATERIALS -->
     <material name="white">
         <color rgba="1 1 1 1 " />
@@ -32,12 +189,17 @@
         <color rgba="1 0 0 1 " />
     </material>
-    <!-- BASE LINK-->
     <link name="base_link">0
     </link>
-    <!-- CHASSIS-->
+    <joint name="base_footprint_joint" type="fixed">
+        <parent link="base_link"/>
+        <child link="base_footprint"/>
+        <origin xyz="0 0 0" rpy="0 0 0"/>
+    </joint>
+    <link name="base_footprint">
+    </link>
     <joint name="chassis_joint" type="fixed">
         <parent link="base_link"/>
         <child link="chassis"/>
-        <origin xyz="0.04 0 ${chassis_height/2 + wheel_radius}" />
+        <origin xyz="-0.08 0 0.06" />
     </joint>
 z
@@ -45,5 +207,5 @@
         <visual>
             <geometry>
-                <box size="0.20 0.20 0.13"/>
+                <box size="${chassis_length} ${chassis_width} ${chassis_height}"/>
             </geometry>
             <material name="black"/>
@@ -52,5 +214,5 @@
             <origin xyz="0 0 0" />
             <geometry>
-                <box size="0.20 0.20 0.13"/>
+                <box size="${chassis_length} ${chassis_width} ${chassis_height}"/>
             </geometry>
         </collision>
@@ -62,5 +224,4 @@
         <material>Gazebo/Black</material>
     </gazebo>
-    <!-- LEFT WHEEL LINK-->
     <joint name="left_wheel_joint" type="continuous">
         <origin xyz="0 ${wheel_offset_y} ${wheel_offset_z}" rpy="-${pi/2} 0 0"/>
@@ -88,5 +249,4 @@
         <material>Gazebo/Blue</material>
     </gazebo>
-    <!-- RIGHT WHEEL LINK-->
     <joint name="right_wheel_joint" type="continuous">
         <origin xyz="0 -${wheel_offset_y} ${wheel_offset_z}" rpy="${pi/2} 0 0"/>
@@ -114,5 +274,4 @@
         <material>Gazebo/Blue</material>
     </gazebo>
-    <!-- CASTER WHEEL-->
     <joint name="caster_wheel_joint" type="fixed">
         <parent link="chassis"/>
@@ -141,3 +300,4 @@
         <mu2 value="0.0001"/>
     </gazebo>
+-->
 </robot>

File: description/ros2_control.xacro (robot description, xacro)
@@ -5,5 +5,5 @@
                 <plugin>gazebo_ros2_control/GazeboSystem</plugin>
             </hardware>
-            <joint name="left_wheel_joint">
+            <joint name="wheel_left_joint">
                 <command_interface name="velocity">
                     <param name="min">-10</param>
@@ -13,5 +13,5 @@
                 <state_interface name="position"/>
             </joint>
-            <joint name="right_wheel_joint">
+            <joint name="wheel_right_joint">
                 <command_interface name="velocity">
                     <param name="min">-10</param>
